File: pcb/alpha_dre_pcb/isio42_pcb.sch (KiCad schematic (older format))
At the start: 106 parts, among them J1 AVR-ISP-6, SW1 SW_Push, U1 ATmega32U4-AU, U2 PRTR5V0U2X, Y1 16MHz

Commit message: Add gerbers
Add gerbers to manufacture the PCB

Add aknowlegment to the readme file
Parts:
- MX1: footprint Button_Switch_Keyboard:SW_Cherry_MX_1.25u_PCB -> isio42_pcb:SW_Cherry_MX_1.00u_PCB_perso
- MX10, MX11, MX12, MX13, MX14, MX15, MX16, MX17, MX18, MX19, MX20, MX21, MX23, MX24, MX25, MX26, MX27, MX28, MX29, MX3, MX30, MX31, MX32, MX33, MX34, MX35, MX36, MX37, MX38, MX39, MX5, MX6, MX7, MX8, MX9: footprint Button_Switch_Keyboard:SW_Cherry_MX_1.00u_PCB -> isio42_pcb:SW_Cherry_MX_1.00u_PCB_perso
- MX2: footprint Button_Switch_Keyboard:SW_Cherry_MX_1.50u_PCB -> isio42_pcb:SW_Cherry_MX_1.50u_PCB_perso
- MX22: footprint Button_Switch_Keyboard:SW_Cherry_MX_6.25u_PCB -> isio42_pcb:SW_Cherry_MX_6.25u_PCB_perso
- MX4, MX42: footprint Button_Switch_Keyboard:SW_Cherry_MX_1.25u_PCB -> isio42_pcb:SW_Cherry_MX_1.25u_PCB_perso
- MX40: footprint Button_Switch_Keyboard:SW_Cherry_MX_ISOEnter_PCB -> isio42_pcb:SW_Cherry_MX_ISOEnter_PCB_perso
- MX41: footprint Button_Switch_Keyboard:SW_Cherry_MX_1.75u_PCB -> isio42_pcb:SW_Cherry_MX_1.75u_PCB_perso
