File: pcb/alpha_dre_pcb/isio42_pcb.kicad_pcb (KiCad board)
At the start: 2 copper layers, 243.7 x 83.3 mm, 108 parts, among them J1 AVR-ISP-6, SW1 SW_Push, U1 ATmega32U4-AU, U2 PRTR5V0U2X, Y1 16MHz

Commit message: Add gerbers
Add gerbers to manufacture the PCB

Add aknowlegment to the readme file
Parts:
- added Ref**: Val**, isio42_pcb:alpha_dre_drawing, F.Cu at (115.9, 99.2)
- MX1: footprint Button_Switch_Keyboard:SW_Cherry_MX_1.25u_PCB -> isio42_pcb:SW_Cherry_MX_1.00u_PCB_perso
- MX10, MX11, MX12, MX13, MX14, MX15, MX16, MX17, MX18, MX19, MX20, MX21, MX23, MX24, MX25, MX26, MX27, MX28, MX29, MX3, MX30, MX31, MX32, MX33, MX34, MX35, MX36, MX37, MX38, MX39, MX5, MX6, MX7, MX8, MX9: footprint Button_Switch_Keyboard:SW_Cherry_MX_1.00u_PCB -> isio42_pcb:SW_Cherry_MX_1.00u_PCB_perso
- MX2: footprint Button_Switch_Keyboard:SW_Cherry_MX_1.50u_PCB -> isio42_pcb:SW_Cherry_MX_1.50u_PCB_perso
- MX22: footprint Button_Switch_Keyboard:SW_Cherry_MX_6.25u_PCB -> isio42_pcb:SW_Cherry_MX_6.25u_PCB_perso
- MX4, MX42: footprint Button_Switch_Keyboard:SW_Cherry_MX_1.25u_PCB -> isio42_pcb:SW_Cherry_MX_1.25u_PCB_perso
- MX40: footprint Button_Switch_Keyboard:SW_Cherry_MX_ISOEnter_PCB -> isio42_pcb:SW_Cherry_MX_ISOEnter_PCB_perso
- MX41: footprint Button_Switch_Keyboard:SW_Cherry_MX_1.75u_PCB -> isio42_pcb:SW_Cherry_MX_1.75u_PCB_perso
- moved Ref** 132.7 mm to (248.4, 104.8)
- moved MX1 2.38 mm to (35.7, 36.5)
- moved G*** 0.79 mm to (176.2, 95.2)
Routing:
- net RESET: track 126.9 -> 134.9 mm
- net Net-(D23-Pad2): track 0.00 -> 6.03 mm
- net +5V: track 211.6 -> 207.0 mm
- net GND: track 233.1 -> 237.4 mm, vias 15 -> 24
- net Earth: track 22.3 -> 25.4 mm, vias 0 -> 1
- net COL11: track 157.3 -> 155.1 mm
- net SCK: track 121.6 -> 119.4 mm
- net Net-(D1-Pad2): track 8.33 -> 6.77 mm
- net ROW3: track 292.3 -> 290.9 mm
- net Net-(R5-Pad1): track 6.26 -> 5.04 mm
- net COL0: track 213.4 -> 214.4 mm
- net MISO: track 107.4 -> 107.9 mm
- net COL5: track 99.2 -> 98.7 mm

Commit message: Update renders
Add holes for the tray mounted version (update gerbers)

Add new rends with precise dimensions
Parts:
- moved U2 4.96 mm to (143.1, 44.6)
- moved R5 3.85 mm to (151.6, 37.3), turned to 90 degrees
- moved F1 3.30 mm to (138.1, 47.5)
- moved R6 2.67 mm to (140.7, 39.7)
- moved USB1 1.35 mm to (143.7, 26.2)
- moved FB1 1.12 mm to (134.7, 33.3)
Routing:
- net Earth: track 25.4 -> 0.00 mm
- net GND: track 237.4 -> 256.0 mm, vias 24 -> 27
- net ROW3: track 290.9 -> 298.1 mm
- net +5V: track 207.0 -> 201.4 mm
- net COL6: track 82.4 -> 87.5 mm
- net Net-(R5-Pad1): track 5.04 -> 9.15 mm
- net VCC: track 21.7 -> 24.3 mm
- net ROW1: track 267.3 -> 269.6 mm
- net COL0: track 214.4 -> 216.7 mm
- net D+: track 78.1 -> 76.4 mm
- net Net-(R6-Pad1): track 4.42 -> 5.60 mm
- net D-: track 75.4 -> 74.4 mm
- net COL8: track 97.5 -> 98.2 mm
Other:
- board size 243.7 x 83.3 mm -> 243.7 x 82.5 mm

Commit message: Added gerbers and renders
Parts:
- removed the Ref** at (248.4, 104.8)
- added Ref**: Val**, isio42_pcb:info_drawing, B.Cu at (90.5, 104.8)
- moved Ref** 134.0 mm to (249.2, 112.7)
- moved C5 6.20 mm to (189.2, 91.3)
- moved D1 5.84 mm to (31.8, 46.8), turned to 180 degrees
- moved C4 4.83 mm to (189.2, 99.2)
- moved C2 3.97 mm to (189.2, 88.1)
- moved D21 3.17 mm to (119.9, 83.3)
- moved D25 2.38 mm to (138.9, 83.4)
- moved Y1 1.77 mm to (188.9, 95.2), turned to 180 degrees
- moved G*** 0.79 mm to (175.4, 95.2)
- moved U2 0.79 mm to (143.9, 44.6)
Routing:
- net GND: track 256.0 -> 239.9 mm, vias 27 -> 31
- net ROW2: track 248.7 -> 258.1 mm
- net ROW0: track 274.0 -> 266.8 mm, vias 7 -> 6
- net COL8: track 98.2 -> 103.8 mm
- net +5V: track 201.4 -> 205.5 mm
- net XTAL2: track 14.1 -> 10.7 mm
- net COL11: track 154.8 -> 156.9 mm
- net XTAL1: track 15.2 -> 13.2 mm
- net Net-(D21-Pad2): track 6.82 -> 8.64 mm
- net RESET: track 134.9 -> 136.3 mm
- net Net-(D1-Pad2): track 6.77 -> 8.11 mm
- net ROW3: track 298.1 -> 299.2 mm
- net COL9: track 112.5 -> 113.5 mm
- net COL10: track 134.7 -> 135.8 mm
- net Net-(D25-Pad2): track 7.62 -> 8.64 mm
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Other:
- outline, holes or cut-outs redrawn

Commit message: Update case files, pcb drawings
Parts:
- removed the Ref** at (90.5, 104.8)
- removed the Ref** at (249.2, 112.7)
- added Ref**: Val**, isio42_pcb:escargot_design, B.Cu at (157.2, 89.7)
- added Ref**: Val**, isio42_pcb:info_design, F.Cu at (104.8, 101.6)
- added Ref**: Val**, isio42_pcb:alpha_dre_design, F.Cu at (115.9, 89.7)
- moved D31 3.97 mm to (180.2, 72.2), turned to 0 degrees
Routing:
- net ROW2: track 258.1 -> 274.0 mm, vias 2 -> 3
- net D+: track 75.8 -> 80.4 mm
- net D-: track 73.8 -> 78.4 mm
- net COL0: track 216.7 -> 214.1 mm
- net COL9: track 113.5 -> 115.8 mm
- net ROW0: track 266.8 -> 268.7 mm
- net COL7: track 73.6 -> 75.2 mm
- net Net-(D31-Pad2): track 4.35 -> 5.04 mm
